File: bottom.kicad_sch (KiCad schematic)
At the start: 0 parts

Commit message: stuff
Parts:
- added C34: 1uF, symbol Device:C
- added C35: 4.7uF, symbol Device:C
- added C36, C37, C38, C40, C41, C42, C44, C45, C48, C50, C51: 100n, symbol Device:C
- added C39, C43, C46, C47, C49: 2.2uF, symbol Device:C
- added C52: 10uF, symbol Device:C
- added D23: 1SMB5949BT3G 100V, symbol Device:D
- added D24, D25, D8, D9: D, symbol Device:D
- added D26: 6.2V, symbol Device:D_Zener
- added L2: L, symbol Device:L
- added Q17, Q18, Q19, Q20, Q21, Q22, Q23, Q24, Q25, Q26: Q_Dual_NMOS_G1S2G2D2S1D1, symbol Transistor_FET:Q_Dual_NMOS_G1S2G2D2S1D1
- added Q27, Q28, Q29, Q30: SI7846DP, symbol Simulation_SPICE:NMOS
- added R38, R39, R41, R44, R47: 100k, symbol Device:R
- added R40, R45, R46: R, symbol Device:R
- added R42: 0.033, symbol Device:R
- added R43: 10k, symbol Device:R
- added R48: 0.01R, symbol Device:R
- added U10: ~, symbol samir:750311492
- added U7: ~, symbol samir:EMB1428QSQ
- added U8: ~, symbol samir:EMB1412MY
- added U9: ~, symbol samir:EMB1499QMH
Connections:
- new net: C51.2, Q28.1 (D)
- new net: C48.2, D9.2 (A), Q28.2 (G), R43.2
- new net: C52.1, D25.2 (A), D26.1 (K), L2.2, Q25.4 (D), Q25.6 (D), R39.2
- new net: Q20.2 (S), Q20.5 (S), U7.9 (S4)
- new net: Q20.1 (G), Q20.3 (G), U7.10 (G4)
- new net: Q27.2 (G), R40.2, R41.1
- new net: Q27.3 (S), R41.2, R42.2
- new net: Q21.2 (S), Q21.5 (S), U7.11 (S3)
- new net: Q21.1 (G), Q21.3 (G), U7.12 (G3)
- new net: Q23.2 (S), Q23.5 (S), U7.16 (S1)
- new net: Q23.1 (G), Q23.3 (G), U7.17 (G1)
- new net: Q17.2 (S), Q17.5 (S), U7.3 (S7)
- new net: Q17.1 (G), Q17.3 (G), U7.4 (G7)
- new net: C51.1, D23.1 (K), Q27.1 (D), U10.1
- new net: D24.2 (A), L2.1, Q30.1 (D), U10.7, U10.8
- new net: R39.1, U9.2 (CELLPLUS)
- new net: Q30.2 (G), R46.1, R47.2
- new net: Q29.3 (S), Q30.3 (S), R44.1, R47.1, R48.2, U9.1 (VSENSE_HS)
- new net: C38.2, U7.47 (CEXT1)
- new net: Q18.1 (G), Q18.3 (G), U7.6 (G6)
- new net: Q18.2 (S), Q18.5 (S), U7.5 (S6)
- new net: C39.1, R38.2, U9.6 (VSET)
- new net: C48.1, U8.7 (OUT)
- new net: Q19.1 (G), Q19.3 (G), U7.8 (G5)
- new net: Q19.2 (S), Q19.5 (S), U7.7 (S5)
- new net: Q29.2 (G), R44.2, R45.1
- new net: R45.2, U9.25 (GATE_HS2)
- new net: C44.2, C46.2, U9.24 (PGNDF), U9.27 (GNDF)
- new net: C36.2, D8.1 (K), U7.45 (VDD_CP)
- new net: Q22.2 (S), Q22.5 (S), U7.14 (S2)
- new net: Q22.1 (G), Q22.3 (G), U7.15 (G2)
- new net: Q24.2 (S), Q24.5 (S), U7.18 (S0)
- new net: Q24.1 (G), Q24.3 (G), U7.19 (G0)
- new net: U7.20 (FAULT_2), U9.14 (FAULT2)
- new net: U7.21 (FAULT_1), U9.13 (FAULT1)
- new net: U7.22 (FAULT_0), U9.12 (FAULT0)
- new net: U7.23 (DONE), U9.11 (DONE)
- new net: U7.24 (~{DIR_RT}), U9.10 (DIR_RT)
- new net: U7.25 (DIR), U9.9 (DIR)
- new net: U7.26 (EN), U9.8 (EN)
- new net: C37.2, U7.46 (CEXT2)
- new net: D24.1 (K), D25.1 (K)
- new net: R46.2, U9.23 (GATE_HS1)
- new net: Q29.1 (D), U10.11, U10.12
- new net: U10.10, U10.9
- new net: U10.2, U10.3
- new net +12V: C35.2, C40.1, C43.1, C44.1, C45.1, C46.1, C47.1, R40.1, U7.2 (VDDP), U7.34 (VDD_12V), U8.4 (IN), U8.6 (VCC), U9.16 (VINA), U9.19 (GATE_LS), U9.21 (VINP), U9.22 (PVINF), U9.28 (VINF)
- new net +3.3V: C42.1, U7.32 (VDD_IO)
- new net +5V: C41.1, U7.33 (VDD_5V)
- new net +VIN: C34.1, C36.1, C37.1, C38.1, D8.2 (A), U7.48 (VSTACK)
- new net BAT.BAT10: Q21.6 (D)
- new net BAT.BAT11: Q20.6 (D)
- new net BAT.BAT12: Q19.6 (D)
- new net BAT.BAT13: Q18.6 (D)
- new net BAT.BAT14: Q17.6 (D)
- new net BAT.BAT7: Q24.6 (D)
- new net BAT.BAT8: Q23.6 (D)
- new net BAT.BAT9: Q22.6 (D)
- new net CS: U7.30 (~{CS})
- new net G10: Q25.1 (G), U7.40 (G10)
- new net G11: Q25.3 (G), U7.38 (G11)
- new net G8: Q26.1 (G), U7.44 (G8)
- new net G9: Q26.3 (G), U7.42 (G9)
- new net GND: C34.2, C35.1, C39.2, C40.2, C41.2, C42.2, C43.2, C45.2, C47.2, C49.2, C50.2, C52.2, D23.2 (A), D26.2 (A), D9.1 (K), Q26.2 (S), Q26.5 (S), Q28.3 (S), R42.1, R43.1, R48.1, U7.1 (GNDP), U7.13 (GND), U7.36 (GND), U7.41 (S9), U7.43 (S8), U7.49 (DAP), U8.1 (IN_REF), U8.3 (VEE), U8.9 (DAP), U9.17 (GNDA), U9.20 (GNDP), U9.29 (DAP), U9.3 (LOR), U9.4 (TM), U9.5 (GNDA), U9.7 (WDOR)
- new net SPI.CLK: U7.27 (SCL_C)
- new net SPI.MISO: U7.29 (SDO)
- new net SPI.MOSI: U7.28 (SDI)
- new net VIN: C49.1, C50.1, U10.4
- new net VREF: R38.1
- new net even: Q18.4 (D), Q20.4 (D), Q22.4 (D), Q24.4 (D), Q25.5 (S), Q26.6 (D), U7.39 (S10)
- new net odd: Q17.4 (D), Q19.4 (D), Q21.4 (D), Q23.4 (D), Q25.2 (S), Q26.4 (D), U7.37 (S11)
- no-connect marks 0 -> 7
Other:
- note added: "EMB1412M"
- note added: "EMB1428QSQ"
- note added: "EMB1499QMH"
- title: (none) -> Bottom
