File: engine.kicad_sch (KiCad schematic)
At the start: 55 parts, among them Q1 Q_Dual_NMOS_G1S2G2D2S1D1, Q10 Q_Dual_NMOS_G1S2G2D2S1D1, Q11 SI7846DP, Q12 SI7846DP, Q13 SI7846DP, Q14 SI7846DP, Q2 Q_Dual_NMOS_G1S2G2D2S1D1, Q3 Q_Dual_NMOS_G1S2G2D2S1D1, Q4 Q_Dual_NMOS_G1S2G2D2S1D1, Q5 Q_Dual_NMOS_G1S2G2D2S1D1, Q6 Q_Dual_NMOS_G1S2G2D2S1D1, Q7 Q_Dual_NMOS_G1S2G2D2S1D1, Q8 Q_Dual_NMOS_G1S2G2D2S1D1, Q9 Q_Dual_NMOS_G1S2G2D2S1D1

Commit message: stuff
Connections:
- net GND: now also Q10.2 (S), Q10.5 (S), U1.41 (S9), U1.43 (S8)
- net PLUS: now also Q9.4 (D), Q9.6 (D)
Changed lines of the file:
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@@
 	)
 	(junction
+		(at 241.3 63.5)
+		(diameter 0)
+		(color 0 0 0 0)
+	)
+	(junction
 		(at 321.31 180.34)
 		(diameter 0)
@@
 	)
 	(junction
+		(at 241.3 49.53)
+		(diameter 0)
+		(color 0 0 0 0)
+	)
+	(junction
 		(at 264.16 140.97)
 		(diameter 0)
@@
 	)
 	(junction
+		(at 241.3 35.56)
+		(diameter 0)
+		(color 0 0 0 0)
+	)
+	(junction
 		(at 264.16 233.68)
 		(diameter 0)
@@
 	)
 	(junction
-		(at 233.68 63.5)
-		(diameter 0)
-		(color 0 0 0 0)
-	)
-	(junction
 		(at 55.88 40.64)
 		(diameter 0)
@@
 	(wire
 		(pts
+			(xy 241.3 49.53) (xy 245.11 49.53)
+		)
+		(stroke
+			(width 0)
+			(type default)
+		)
+	)
+	(wire
+		(pts
 			(xy 53.34 162.56) (xy 60.96 162.56)
 		)
@@
 	(wire
 		(pts
+			(xy 241.3 35.56) (xy 245.11 35.56)
+		)
+		(stroke
+			(width 0)
+			(type default)
+		)
+	)
+	(wire
+		(pts
 			(xy 233.68 172.72) (xy 233.68 165.1)
 		)
@@
 	(wire
 		(pts
-			(xy 233.68 68.58) (xy 233.68 63.5)
+			(xy 241.3 68.58) (xy 241.3 63.5)
 		)
 		(stroke
@@
 	(wire
 		(pts
-			(xy 233.68 63.5) (xy 231.14 63.5)
+			(xy 231.14 63.5) (xy 241.3 63.5)
 		)
 		(stroke
@@
 	(wire
 		(pts
-			(xy 241.3 63.5) (xy 233.68 63.5)
-		)
-		(stroke
-			(width 0)
-			(type default)
-		)
-	)
-	(wire
-		(pts
 			(xy 321.31 166.37) (xy 321.31 127)
 		)
@@
 	(wire
 		(pts
-			(xy 207.01 68.58) (xy 233.68 68.58)
+			(xy 207.01 68.58) (xy 241.3 68.58)
 		)
 		(stroke
@@
 		)
 	)
+	(hierarchical_label "MINUS"
+		(shape input)
+		(at 245.11 49.53 0)
+		(effects
+			(font
+				(size 1.27 1.27)
+			)
+			(justify left)
+		)
+	)
 	(hierarchical_label "PLUS"
 		(shape input)
@@
 		)
 	)
+	(hierarchical_label "PLUS"
+		(shape input)
+		(at 245.11 35.56 0)
+		(effects
+			(font
+				(size 1.27 1.27)
+			)
+			(justify left)
+		)
+	)

Commit message: stuff
Connections:
- net GND: now also U1.13 (GND)
- net SPI.CLK: now reaches U1.27 (SCL_C)
- net SPI.MOSI: now reaches U1.28 (SDI)
- net SPI.MISO: now reaches U1.29 (SDO)
- net CS: now reaches U1.30 (~{CS})
- net PLUS: no longer names the net of C19.1, D5.2 (A), D6.1 (K), L1.2, Q9.4 (D), Q9.6 (D), R10.2
- no-connect marks 6 -> 7
Other:
- note added: "EMB1412M"
- note added: "EMB1428QSQ"
- note added: "EMB1499QMH"
- moved on the sheet: C1, C16, C17, C2, C3, C4, C5, C6, C7, C8, D1, D3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
